File: OSD19001_BRK_X2.kicad_pcb (KiCad board)
At the start: 4 copper layers, 45.7 x 76.2 mm, 162 parts, among them J1 UJ2-MIBH2-4-SMT, J2 104031-0811, U1 OSD32MP157C-512M-BAA, Y1 32.768KHz

Commit message: Renamed PA01=>PA1, etc (for PA/PB/PC/PD01-09) on PCB
Parts:
- renumbered PA01 to PA1, PA02 to PA2, PA03 to PA3, PA04 to PA4, PA05 to PA5, PA06 to PA6, PA07 to PA7, PA08 to PA8, PA09 to PA9, PB01 to PB1, PB02 to PB2, PB03 to PB3, PB04 to PB4, PB05 to PB5, PB06 to PB6, PB07 to PB7, PB08 to PB8, PB09 to PB9, PC01 to PC1, PC02 to PC2, PC03 to PC3, PC04 to PC4, PC05 to PC5, PC06 to PC6, PC08 to PC8, PC09 to PC9, PD01 to PD1, PD02 to PD2, PD03 to PD3, PD04 to PD4, PD05 to PD5, PD06 to PD6, PD07 to PD7, PD08 to PD8, PD09 to PD9

Commit message: Appened 1 to  PTXD, PRXD, PGND to match schematic
Parts:
- renumbered PGND to PGND1, PRXD to PRXD1, PTXD to PTXD1
Changed lines of the file:
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@@
   (footprint "ACWPrimitives.IntLib:LP_TESTPOINT_TH" locked (layer "F.Cu")
     (at 148.501099 118.973597 -90)
-    (fp_text reference "PRXD" (at -1.2065 0.4445 unlocked) (layer "F.SilkS") hide
+    (fp_text reference "PRXD1" (at -1.2065 0.4445 unlocked) (layer "F.SilkS") hide
       (effects (font (size 1.524 1.524) (thickness 0.254)) (justify left bottom))
     )
@@
   (footprint "ACWPrimitives.IntLib:LP_TESTPOINT_TH" locked (layer "F.Cu")
     (at 145.961099 118.973597 -90)
-    (fp_text reference "PGND" (at -1.235944 7.184487 unlocked) (layer "F.SilkS") hide
+    (fp_text reference "PGND1" (at -1.235944 7.184487 unlocked) (layer "F.SilkS") hide
       (effects (font (size 1.524 1.524) (thickness 0.254)) (justify left bottom))
     )
@@
   (footprint "ACWPrimitives.IntLib:LP_TESTPOINT_TH" locked (layer "F.Cu")
     (at 151.041099 118.973597 -90)
-    (fp_text reference "PTXD" (at 3.8735 -9.4615 unlocked) (layer "F.SilkS") hide
-      (effects (font (size 1.524 1.524) (thickness 0.254)) (justify left bottom))
-    )
+    (fp_text reference "PTXD1" (at 3.8735 -9.4615 unlocked) (layer "F.SilkS") hide
+      (effects (font (size 1.524 1.524) (thickness 0.254)) (justify left bottom))
+    )

Commit message: Missed PC07=>PC7 on PCB
Parts:
- renumbered PC07 to PC7
Changed lines of the file:
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@@
   (footprint "ACWPrimitives.IntLib:LP_TESTPOINT_TH" (layer "F.Cu")
     (at 167.551099 83.413597 90)
-    (fp_text reference "PC07" (at 1.636278 -0.617807 unlocked) (layer "F.SilkS") hide
+    (fp_text reference "PC7" (at 1.636278 -0.617807 unlocked) (layer "F.SilkS") hide
       (effects (font (size 1.524 1.524) (thickness 0.254)) (justify left bottom))
     )

Commit message: Updated PCB from schematic. Saved log
Connections:
- net ANA0 renamed /SH_OSD19001_BREAKOUTS/ANA0
- net ANA1 renamed /SH_OSD19001_BREAKOUTS/ANA1
- net BOOT0 renamed /SH_OSD19001_CORE/BOOT0
- net BOOT1 renamed /SH_OSD19001_CORE/BOOT1
- net BOOT2 renamed /SH_OSD19001_CORE/BOOT2
- net EEPROM_WP renamed /SH_OSD19001_CORE/EEPROM_WP
- net NetC10_2 renamed Net-(C10-Pad2)
- net NetC3_1 renamed Net-(C3-Pad1)
- net NetC4_1 renamed Net-(C4-Pad1)
- net NetD1_1 renamed Net-(D1-Pad1)
- net NetD1_2 renamed Net-(D1-Pad2)
- net NetD2_1 renamed Net-(D2-Pad1)
- net NetD2_2 renamed Net-(D2-Pad2)
- net NetD3_1 renamed Net-(D3-Pad1)
- net NetD3_2 renamed Net-(D3-Pad2)
- net NetR8_1 renamed Net-(R8-Pad1)
- net NetU1_K1 renamed Net-(U1-PadK1)
- net NetU1_M1 renamed Net-(U1-PadM1)
- net PA1 renamed /SH_OSD19001_BREAKOUTS/PA1
- net PA14 renamed /SH_OSD19001_BREAKOUTS/PA14
- net PA15 renamed /SH_OSD19001_BREAKOUTS/PA15
- net PA2 renamed /SH_OSD19001_BREAKOUTS/PA2
- net PA3 renamed /SH_OSD19001_BREAKOUTS/PA3
- net PA4 renamed /SH_OSD19001_BREAKOUTS/PA4
- net PA5 renamed /SH_OSD19001_BREAKOUTS/PA5
- net PA6 renamed /SH_OSD19001_BREAKOUTS/PA6
- net PA7 renamed /SH_OSD19001_BREAKOUTS/PA7
- net PA9 renamed /SH_OSD19001_BREAKOUTS/PA9
- net PB0 renamed /SH_OSD19001_BREAKOUTS/PB0
- net PB1 renamed /SH_OSD19001_BREAKOUTS/PB1
- net PB10 renamed /SH_OSD19001_BREAKOUTS/PB10
- net PB11 renamed /SH_OSD19001_BREAKOUTS/PB11
- net PB12 renamed /SH_OSD19001_BREAKOUTS/PB12
- net PB13 renamed /SH_OSD19001_BREAKOUTS/PB13
- net PB14 renamed /SH_OSD19001_BREAKOUTS/PB14
- net PB15 renamed /SH_OSD19001_BREAKOUTS/PB15
- net PB3 renamed /SH_OSD19001_BREAKOUTS/PB3
- net PB4 renamed /SH_OSD19001_BREAKOUTS/PB4
- net PB5 renamed /SH_OSD19001_BREAKOUTS/PB5
- net PB6 renamed /SH_OSD19001_BREAKOUTS/PB6
- net PB7 renamed /SH_OSD19001_BREAKOUTS/PB7
- net PB8 renamed /SH_OSD19001_BREAKOUTS/PB8
- net PB9 renamed /SH_OSD19001_BREAKOUTS/PB9
- net PC0 renamed /SH_OSD19001_BREAKOUTS/PC0
- net PC1 renamed /SH_OSD19001_BREAKOUTS/PC1
- net PC2 renamed /SH_OSD19001_BREAKOUTS/PC2
- net PC3 renamed /SH_OSD19001_BREAKOUTS/PC3
- net PC4 renamed /SH_OSD19001_BREAKOUTS/PC4
- net PC5 renamed /SH_OSD19001_BREAKOUTS/PC5
- net PC7 renamed /SH_OSD19001_BREAKOUTS/PC7
- net PD0 renamed /SH_OSD19001_BREAKOUTS/PD0
- net PD1 renamed /SH_OSD19001_BREAKOUTS/PD1
- net PD10 renamed /SH_OSD19001_BREAKOUTS/PD10
- net PD11 renamed /SH_OSD19001_BREAKOUTS/PD11
- net PD12 renamed /SH_OSD19001_BREAKOUTS/PD12
- net PD13 renamed /SH_OSD19001_BREAKOUTS/PD13
- net PD14 renamed /SH_OSD19001_BREAKOUTS/PD14
- net PD15 renamed /SH_OSD19001_BREAKOUTS/PD15
- net PD3 renamed /SH_OSD19001_BREAKOUTS/PD3
- net PD4 renamed /SH_OSD19001_BREAKOUTS/PD4
- net PD5 renamed /SH_OSD19001_BREAKOUTS/PD5
- net PD6 renamed /SH_OSD19001_BREAKOUTS/PD6
- net PD7 renamed /SH_OSD19001_BREAKOUTS/PD7
- net PD8 renamed /SH_OSD19001_BREAKOUTS/PD8
- net PD9 renamed /SH_OSD19001_BREAKOUTS/PD9
- net PE0 renamed /SH_OSD19001_BREAKOUTS/PE0
- net PE1 renamed /SH_OSD19001_BREAKOUTS/PE1
- net PE11 renamed /SH_OSD19001_BREAKOUTS/PE11
- net PE12 renamed /SH_OSD19001_BREAKOUTS/PE12
- net PE13 renamed /SH_OSD19001_BREAKOUTS/PE13
- net PE14 renamed /SH_OSD19001_BREAKOUTS/PE14
- net PE15 renamed /SH_OSD19001_BREAKOUTS/PE15
- net PE2 renamed /SH_OSD19001_BREAKOUTS/PE2
- net PE3 renamed /SH_OSD19001_BREAKOUTS/PE3
- net PE5 renamed /SH_OSD19001_BREAKOUTS/PE5
- net PE6 renamed /SH_OSD19001_BREAKOUTS/PE6
- net PF0 renamed /SH_OSD19001_BREAKOUTS/PF0
- net PF1 renamed /SH_OSD19001_BREAKOUTS/PF1
- net PF11 renamed /SH_OSD19001_BREAKOUTS/PF11
- net PF12 renamed /SH_OSD19001_BREAKOUTS/PF12
- net PF13 renamed /SH_OSD19001_BREAKOUTS/PF13
- net PF14 renamed /SH_OSD19001_BREAKOUTS/PF14
- net PF15 renamed /SH_OSD19001_BREAKOUTS/PF15
- net PF3 renamed /SH_OSD19001_BREAKOUTS/PF3
- net PF4 renamed /SH_OSD19001_BREAKOUTS/PF4
- net PF5 renamed /SH_OSD19001_BREAKOUTS/PF5
- net PF6 renamed /SH_OSD19001_BREAKOUTS/PF6
- net PG0 renamed /SH_OSD19001_BREAKOUTS/PG0
- net PG1 renamed /SH_OSD19001_BREAKOUTS/PG1
- net PG12 renamed /SH_OSD19001_BREAKOUTS/PG12
- net PG13 renamed /SH_OSD19001_BREAKOUTS/PG13
- net PG14 renamed /SH_OSD19001_BREAKOUTS/PG14
- net PG15 renamed /SH_OSD19001_BREAKOUTS/PG15
- net PG2 renamed /SH_OSD19001_BREAKOUTS/PG2
- net PG3 renamed /SH_OSD19001_BREAKOUTS/PG3
- net PG4 renamed /SH_OSD19001_BREAKOUTS/PG4
- net PG5 renamed /SH_OSD19001_BREAKOUTS/PG5
- net PG6 renamed /SH_OSD19001_BREAKOUTS/PG6
- net PH10 renamed /SH_OSD19001_BREAKOUTS/PH10
- net PH11 renamed /SH_OSD19001_BREAKOUTS/PH11
- net PH12 renamed /SH_OSD19001_BREAKOUTS/PH12
- net PH13 renamed /SH_OSD19001_BREAKOUTS/PH13
- net PH14 renamed /SH_OSD19001_BREAKOUTS/PH14
- net PH15 renamed /SH_OSD19001_BREAKOUTS/PH15
- net PH4 renamed /SH_OSD19001_BREAKOUTS/PH4
- net PH5 renamed /SH_OSD19001_BREAKOUTS/PH5
- net PH8 renamed /SH_OSD19001_BREAKOUTS/PH8
- net PH9 renamed /SH_OSD19001_BREAKOUTS/PH9
- net PI0 renamed /SH_OSD19001_BREAKOUTS/PI0
- net PI1 renamed /SH_OSD19001_BREAKOUTS/PI1
- net PI2 renamed /SH_OSD19001_BREAKOUTS/PI2
- net PI3 renamed /SH_OSD19001_BREAKOUTS/PI3
- net PI4 renamed /SH_OSD19001_BREAKOUTS/PI4
- net PI5 renamed /SH_OSD19001_BREAKOUTS/PI5
- net PI6 renamed /SH_OSD19001_BREAKOUTS/PI6
- net PI7 renamed /SH_OSD19001_BREAKOUTS/PI7
- net PZ0 renamed /SH_OSD19001_BREAKOUTS/PZ0
- net PZ1 renamed /SH_OSD19001_BREAKOUTS/PZ1
- net PZ2 renamed /SH_OSD19001_BREAKOUTS/PZ2
- net PZ3 renamed /SH_OSD19001_BREAKOUTS/PZ3
- net PZ4 renamed /SH_OSD19001_BREAKOUTS/PZ4
- net PZ5 renamed /SH_OSD19001_BREAKOUTS/PZ5
- net SDMMC1_CK renamed /SH_OSD19001_BREAKOUTS/SDMMC1_CK
- net SDMMC1_CMD renamed /SH_OSD19001_BREAKOUTS/SDMMC1_CMD
- net SDMMC1_D0 renamed /SH_OSD19001_BREAKOUTS/SDMMC1_D0
- net SDMMC1_D1 renamed /SH_OSD19001_BREAKOUTS/SDMMC1_D1
- net SDMMC1_D2 renamed /SH_OSD19001_BREAKOUTS/SDMMC1_D2
- net SDMMC1_D3 renamed /SH_OSD19001_BREAKOUTS/SDMMC1_D3
- net SWCLK/TCK renamed /SH_OSD19001_CORE/SWCLK/TCK
- net SWDIO/TMS renamed /SH_OSD19001_CORE/SWDIO/TMS
- net SWO/TDO renamed /SH_OSD19001_CORE/SWO/TDO
- net TDI renamed /SH_OSD19001_CORE/TDI
- net UART4_RX renamed /SH_OSD19001_BREAKOUTS/UART4_RX
- net UART4_TX renamed /SH_OSD19001_BREAKOUTS/UART4_TX
- net USB1_D_N renamed /SH_OSD19001_BREAKOUTS/USB1_D_N
- net USB1_D_P renamed /SH_OSD19001_BREAKOUTS/USB1_D_P
- net USB2_D_N renamed /SH_OSD19001_USB/USB2_D_N
- net USB2_D_P renamed /SH_OSD19001_USB/USB2_D_P
- net VWALLP renamed /SH_OSD19001_USB/VWALLP
- net \LED1_GRN renamed /SH_OSD19001_BREAKOUTS/\LED1_GRN
- net \LED1_RED renamed /SH_OSD19001_BREAKOUTS/\LED1_RED
- net \LED2_GRN renamed /SH_OSD19001_BREAKOUTS/\LED2_GRN
- net \LED2_RED renamed /SH_OSD19001_BREAKOUTS/\LED2_RED
- net \PONKEY renamed /SH_OSD19001_BREAKOUTS/\PONKEY
- net \RESET renamed /SH_OSD19001_BREAKOUTS/\RESET
- net \SDDET renamed /SH_OSD19001_BREAKOUTS/\SDDET
- net \TRST renamed /SH_OSD19001_CORE/\TRST
- TP1 pad 7: (no net) -> unconnected-(TP1-Pad7)
- U1 pad A3: (no net) -> unconnected-(U1-PadA3)
- U1 pad B13: (no net) -> unconnected-(U1-PadB13)
- U1 pad B4: (no net) -> unconnected-(U1-PadB4)
- U1 pad B5: (no net) -> unconnected-(U1-PadB5)
- U1 pad C13: (no net) -> unconnected-(U1-PadC13)
- U1 pad C18: (no net) -> unconnected-(U1-PadC18)
- U1 pad C4: (no net) -> unconnected-(U1-PadC4)
- U1 pad C5: (no net) -> unconnected-(U1-PadC5)
- U1 pad D10: (no net) -> unconnected-(U1-PadD10)
- U1 pad D16: (no net) -> unconnected-(U1-PadD16)
- U1 pad D17: (no net) -> unconnected-(U1-PadD17)
- U1 pad D18: (no net) -> unconnected-(U1-PadD18)
- U1 pad D5: (no net) -> unconnected-(U1-PadD5)
- U1 pad D6: (no net) -> unconnected-(U1-PadD6)
- U1 pad D7: (no net) -> unconnected-(U1-PadD7)
- U1 pad D8: (no net) -> unconnected-(U1-PadD8)
- U1 pad D9: (no net) -> unconnected-(U1-PadD9)
- U1 pad E16: (no net) -> unconnected-(U1-PadE16)
- U1 pad E17: (no net) -> unconnected-(U1-PadE17)
- U1 pad G16: (no net) -> unconnected-(U1-PadG16)
- U1 pad G17: (no net) -> unconnected-(U1-PadG17)
- U1 pad G18: (no net) -> unconnected-(U1-PadG18)
- U1 pad G8: (no net) -> unconnected-(U1-PadG8)
- U1 pad H12: (no net) -> unconnected-(U1-PadH12)
- U1 pad H16: (no net) -> unconnected-(U1-PadH16)
- U1 pad H4: (no net) -> unconnected-(U1-PadH4)
- U1 pad J12: (no net) -> unconnected-(U1-PadJ12)
- U1 pad J2: (no net) -> unconnected-(U1-PadJ2)
- U1 pad J4: (no net) -> unconnected-(U1-PadJ4)
- U1 pad K12: (no net) -> unconnected-(U1-PadK12)
- U1 pad K6: (no net) -> unconnected-(U1-PadK6)
- U1 pad K8: (no net) -> unconnected-(U1-PadK8)
- U1 pad K9: (no net) -> unconnected-(U1-PadK9)
- U1 pad L12: (no net) -> unconnected-(U1-PadL12)
- U1 pad L16: (no net) -> unconnected-(U1-PadL16)
- U1 pad L17: (no net) -> unconnected-(U1-PadL17)
- U1 pad L18: (no net) -> unconnected-(U1-PadL18)
- U1 pad L3: (no net) -> unconnected-(U1-PadL3)
- U1 pad L6: (no net) -> unconnected-(U1-PadL6)
- U1 pad M16: (no net) -> unconnected-(U1-PadM16)
- U1 pad M17: (no net) -> unconnected-(U1-PadM17)
- U1 pad M6: (no net) -> unconnected-(U1-PadM6)
- U1 pad N16: (no net) -> unconnected-(U1-PadN16)
- U1 pad N17: (no net) -> unconnected-(U1-PadN17)
- U1 pad N18: (no net) -> unconnected-(U1-PadN18)
- U1 pad N4: (no net) -> unconnected-(U1-PadN4)
- U1 pad P10: (no net) -> unconnected-(U1-PadP10)
- U1 pad P16: (no net) -> unconnected-(U1-PadP16)
- U1 pad P17: (no net) -> unconnected-(U1-PadP17)
- U1 pad P18: (no net) -> unconnected-(U1-PadP18)
- U1 pad P9: (no net) -> unconnected-(U1-PadP9)
- U1 pad R10: (no net) -> unconnected-(U1-PadR10)
- U1 pad R17: (no net) -> unconnected-(U1-PadR17)
- U1 pad R18: (no net) -> unconnected-(U1-PadR18)
- U1 pad R4: (no net) -> unconnected-(U1-PadR4)
- U1 pad R5: (no net) -> unconnected-(U1-PadR5)
- U1 pad R6: (no net) -> unconnected-(U1-PadR6)
- U1 pad R7: (no net) -> unconnected-(U1-PadR7)
- U1 pad R8: (no net) -> unconnected-(U1-PadR8)
- U1 pad R9: (no net) -> unconnected-(U1-PadR9)
- U1 pad T17: (no net) -> unconnected-(U1-PadT17)
- U1 pad T18: (no net) -> unconnected-(U1-PadT18)
