File: OSD19001_CORE.kicad_sch (KiCad schematic)
At the start: 14 parts, among them U1 ${PARTNUMBER}, Y1 ${FREQUENCY}

Commit message: Fixed schematic symbol values: were set to Altium variables
Parts:
- C1, C2: value ${ALTIUM_VALUE} -> 0.22uF
- C3, C4: value ${ALTIUM_VALUE} -> 12pF
- R7: value ${ALTIUM_VALUE} -> 10K
- R8: value ${ALTIUM_VALUE} -> 330
- S1: value ${PARTNUMBER} -> PTS810
- S2: value ${PARTNUMBER} -> TDA04H0SB1R
- TP1: value ${PARTNUMBER} -> TC2050-IDC-NL
- U1: value ${PARTNUMBER} -> OSD32MP157C-512M-BAA
- Y1: value ${FREQUENCY} -> 32.768KHz
Changed lines of the file:
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@@
       (effects (font (size 1.27 1.27)) (justify left bottom))
     )
-    (property "Value" "${ALTIUM_VALUE}" (id 1) (at 323.85 225.806 0)
+    (property "Value" "330" (id 1) (at 323.85 225.806 0)
       (effects (font (size 1.27 1.27)) (justify left bottom))
     )
@@
       (effects (font (size 1.27 1.27)) (justify left bottom))
     )
-    (property "Value" "${ALTIUM_VALUE}" (id 1) (at 330.708 212.852 0)
+    (property "Value" "10K" (id 1) (at 330.708 212.852 0)
       (effects (font (size 1.27 1.27)) (justify left bottom))
     )
@@
       (effects (font (size 1.27 1.27)) (justify left bottom))
     )
-    (property "Value" "${ALTIUM_VALUE}" (id 1) (at 38.608 85.598 0)
+    (property "Value" "0.22uF" (id 1) (at 38.608 85.598 0)
       (effects (font (size 1.27 1.27)) (justify left bottom))
     )
@@
       (effects (font (size 1.27 1.27)) (justify left bottom))
     )
-    (property "Value" "${ALTIUM_VALUE}" (id 1) (at 51.308 85.598 0)
+    (property "Value" "0.22uF" (id 1) (at 51.308 85.598 0)
       (effects (font (size 1.27 1.27)) (justify left bottom))
     )
@@
       (effects (font (size 1.27 1.27)) (justify left bottom))
     )
-    (property "Value" "${ALTIUM_VALUE}" (id 1) (at 115.062 250.698 0)
+    (property "Value" "12pF" (id 1) (at 115.062 250.698 0)
       (effects (font (size 1.27 1.27)) (justify left bottom))
     )
@@
       (effects (font (size 1.27 1.27)) (justify left bottom))
     )
-    (property "Value" "${ALTIUM_VALUE}" (id 1) (at 147.574 250.698 0)
+    (property "Value" "12pF" (id 1) (at 147.574 250.698 0)
       (effects (font (size 1.27 1.27)) (justify left bottom))
     )
@@
       (effects (font (size 1.27 1.27)) (justify left bottom))
     )
-    (property "Value" "${PARTNUMBER}" (id 1) (at 305.308 225.806 0)
+    (property "Value" "PTS810" (id 1) (at 305.308 225.806 0)
       (effects (font (size 1.27 1.27)) (justify left bottom))
     )
@@
       (effects (font (size 1.27 1.27)) (justify right bottom))
     )
-    (property "Value" "${FREQUENCY}" (id 1) (at 137.922 243.84 0)
+    (property "Value" "32.768KHz" (id 1) (at 137.922 243.84 0)
       (effects (font (size 1.27 1.27)) (justify right top))
     )
@@
       (effects (font (size 1.27 1.27)) (justify left bottom))
     )
-    (property "Value" "${PARTNUMBER}" (id 1) (at 260.604 210.566 0)
+    (property "Value" "TDA04H0SB1R" (id 1) (at 260.604 210.566 0)
       (effects (font (size 1.27 1.27)) (justify left bottom))
     )
@@
       (effects (font (size 1.27 1.27)) (justify left bottom))
     )
-    (property "Value" "${PARTNUMBER}" (id 1) (at 314.96 73.406 0)
+    (property "Value" "OSD32MP157C-512M-BAA" (id 1) (at 314.96 73.406 0)
       (effects (font (size 1.27 1.27)) (justify left bottom))
     )
@@
       (effects (font (size 1.27 1.27)) (justify left bottom))
     )
-    (property "Value" "${PARTNUMBER}" (id 1) (at 178.816 205.74 0)
+    (property "Value" "TC2050-IDC-NL" (id 1) (at 178.816 205.74 0)
       (effects (font (size 1.27 1.27)) (justify left bottom))
     )
@@
       (effects (font (size 1.27 1.27)) (justify left bottom))
     )
-    (property "Value" "${PARTNUMBER}" (id 1) (at 81.026 210.82 0)
+    (property "Value" "OSD32MP157C-512M-BAA" (id 1) (at 81.026 210.82 0)
       (effects (font (size 1.27 1.27)) (justify left bottom))
     )
@@
       (effects (font (size 1.27 1.27)) (justify left bottom))
     )
-    (property "Value" "${PARTNUMBER}" (id 1) (at 255.016 73.66 0)
+    (property "Value" "OSD32MP157C-512M-BAA" (id 1) (at 255.016 73.66 0)
       (effects (font (size 1.27 1.27)) (justify left bottom))
     )
@@
       (effects (font (size 1.27 1.27)) (justify left bottom))
     )
-    (property "Value" "${PARTNUMBER}" (id 1) (at 157.734 73.66 0)
+    (property "Value" "OSD32MP157C-512M-BAA" (id 1) (at 157.734 73.66 0)
       (effects (font (size 1.27 1.27)) (justify left bottom))
     )
@@
       (effects (font (size 1.27 1.27)) (justify left bottom))
     )
-    (property "Value" "${PARTNUMBER}" (id 1) (at 81.026 73.66 0)
-      (effects (font (size 1.27 1.27)) (justify left bottom))
-    )
+    (property "Value" "OSD32MP157C-512M-BAA" (id 1) (at 81.026 73.66 0)
+      (effects (font (size 1.27 1.27)) (justify left bottom))
+    )

Commit message: Corrected title bar text to match online PDF schematic
Other:
- note added: "2"
- note removed: "${#}"
Changed lines of the file:
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@@
+    (stroke (width 0) (type solid) (color 0 0 0 0))
+  )
+  (polyline (pts (xy 375.92 256.54) (xy 375.92 274.32))
+    (stroke (width 0) (type solid) (color 0 0 0 0))
+  )
+  (polyline (pts (xy 375.92 274.32) (xy 259.08 274.32))
     (stroke (width 0) (type solid) (color 0 0 0 0))
   )
@@
     (effects (font (size 1.016 1.016)) (justify left bottom))
   )
-  (text "${#}" (at 307.848 271.78 180)
-    (effects (font (size 1.016 1.016)) (justify left bottom))
+  (text "2" (at 307.848 271.78 180)
+    (effects (font (size 1.016 1.016)) (justify right bottom))
   )
   (text "OF" (at 310.642 271.78 180)
